Commit message: Added Intel RealSense 200 Depth Camera

File: robots_description/models/mbzirc/geometry.xacro (robot description, xacro)
@@ -57,5 +57,5 @@
     <xacro:insert_block name="body_inertia" />
   </xacro:multirotor_base_macro>
-  <xacro:camera_macro
+  <!-- <xacro:camera_macro
     namespace="${namespace}"
     parent_link="base_link"
@@ -74,5 +74,5 @@
     <xacro:insert_block name="camera_cylinder"/>
     <origin xyz="0 0.24 -0.24" rpy="0 1.57 0" />
-  </xacro:camera_macro>
+  </xacro:camera_macro> -->
   <!-- Magnetic gripper -->
   <link name="magnetic_gripper">

File: robots_description/models/mbzirc/model.xacro (robot description, xacro)
@@ -116,8 +116,14 @@
   </xacro:if>
   <!-- Import macro for realsense-RS200 camera-->
-  <!-- <xacro:include filename="$(find realsense_gazebo_plugin)/urdf/realsense-RS200.macro.xacro"/> -->
+  <xacro:include filename="$(find realsense_gazebo_plugin)/urdf/realsense-RS200.macro.xacro"/>
   <!-- Create camera instance -->
-  <!-- <xacro:realsense-rs200 prefix="" parent="base_link">
-      <origin xyz="0.4 0 0.02" rpy="0 0 0" />
-  </xacro:realsense-rs200> -->
+  <xacro:realsense-rs200 prefix="" parent="base_link">
+      <origin xyz="0.22 0 -0.14" rpy="0 0 0" />
+  </xacro:realsense-rs200>
+  <!-- <xacro:vi_sensor_depth_macro
+    namespace="${namespace}"
+    parent_link="base_link"
+    camera_suffix=""
+    frame_rate="30">
+  </xacro:vi_sensor_depth_macro> -->
 </robot>
